Commit message: Base colorida

File: urdf/simple.xacro (robot description, xacro)
@@ -14,5 +14,5 @@
     <origin xyz="0 0 0" rpy="0 0 0"/>
     <geometry>
-      <mesh filename="package://simple_description/meshes/base_link.stl" scale="0.001 0.001 0.001"/>
+      <mesh filename="package://simple_description/meshes/base.dae" scale="0.001 0.001 0.001"/>
     </geometry>
     <material name="silver"/>

Commit message: x

File: urdf/simple.xacro (robot description, xacro)
@@ -14,5 +14,5 @@
     <origin xyz="0 0 0" rpy="0 0 0"/>
     <geometry>
-      <mesh filename="package://simple_description/meshes/base.dae" scale="0.001 0.001 0.001"/>
+      <mesh filename="package://simple_description/meshes/base_link.dae" scale="0.001 0.001 0.001"/>
     </geometry>
     <material name="silver"/>
@@ -34,5 +34,5 @@
     <origin xyz="0.005 0.0515 -0.05045" rpy="0 0 0"/>
     <geometry>
-      <mesh filename="package://simple_description/meshes/shaft1_1.stl" scale="0.001 0.001 0.001"/>
+      <mesh filename="package://simple_description/meshes/shaft1_1.dae" scale="0.001 0.001 0.001"/>
     </geometry>
     <material name="silver"/>
@@ -54,5 +54,5 @@
     <origin xyz="0.005 0.0715 -0.05045" rpy="0 0 0"/>
     <geometry>
-      <mesh filename="package://simple_description/meshes/whell1_1.stl" scale="0.001 0.001 0.001"/>
+      <mesh filename="package://simple_description/meshes/whell1_1.dae" scale="0.001 0.001 0.001"/>
     </geometry>
     <material name="silver"/>
@@ -74,5 +74,5 @@
     <origin xyz="0.005 -0.0515 -0.05045" rpy="0 0 0"/>
     <geometry>
-      <mesh filename="package://simple_description/meshes/shaft2_1.stl" scale="0.001 0.001 0.001"/>
+      <mesh filename="package://simple_description/meshes/shaft2_1.dae" scale="0.001 0.001 0.001"/>
     </geometry>
     <material name="silver"/>
@@ -94,5 +94,5 @@
     <origin xyz="0.005 -0.0715 -0.05045" rpy="0 0 0"/>
     <geometry>
-      <mesh filename="package://simple_description/meshes/whell2_1.stl" scale="0.001 0.001 0.001"/>
+      <mesh filename="package://simple_description/meshes/whell2_1.dae" scale="0.001 0.001 0.001"/>
     </geometry>
     <material name="silver"/>
@@ -114,5 +114,5 @@
     <origin xyz="-0.184 0.037 -0.035" rpy="0 0 0"/>
     <geometry>
-      <mesh filename="package://simple_description/meshes/sensor_1.stl" scale="0.001 0.001 0.001"/>
+      <mesh filename="package://simple_description/meshes/sensor_1.dae" scale="0.001 0.001 0.001"/>
     </geometry>
     <material name="silver"/>
@@ -134,5 +134,5 @@
     <origin xyz="-0.1725 -0.0 -0.0215" rpy="0 0 0"/>
     <geometry>
-      <mesh filename="package://simple_description/meshes/roda2_1.stl" scale="0.001 0.001 0.001"/>
+      <mesh filename="package://simple_description/meshes/roda2_1.dae" scale="0.001 0.001 0.001"/>
     </geometry>
     <material name="silver"/>
@@ -154,5 +154,5 @@
     <origin xyz="-0.1725 0.00675 -0.03" rpy="0 0 0"/>
     <geometry>
-      <mesh filename="package://simple_description/meshes/roda1_1.stl" scale="0.001 0.001 0.001"/>
+      <mesh filename="package://simple_description/meshes/roda1_1.dae" scale="0.001 0.001 0.001"/>
     </geometry>
     <material name="silver"/>
